Commit message: using gpd ros

File: ur5_single_arm_tufts/urdf/ur5_single_arm.urdf.xacro (robot description, xacro)
@@ -18,9 +18,32 @@
     <origin xyz="0.6 0.0 1.8" rpy="0.0 ${pi/2} 0.0" />
   </xacro:kinect-->
+  <!-- depth camera out of robot for kinect v2,
+  the range of detection is from 0.8 m to 4.0 m
+  kinect v2 cannot be installed in wrist, because of the limitation of the range of detection
+  -->
+  <!-- depth camera installed in wrist  -->
+  <!-- minimum depth distance of realsense D435 is 0.11 m  -->
+  <!--      <xacro:kinect_v2  parent="ee_link">-->
+  <!--          <origin xyz="-0.05 0 0.05"-->
+  <!--                  rpy="0 0 0" />-->
+<!--  <xacro:include filename="$(find kinect_v2)/urdf/kinect_v2.urdf.xacro" />-->
+<!--    <xacro:kinect_v2  parent="world">-->
+<!--        <origin xyz="0.6 0 1.00"-->
+<!--                rpy="0 1.57 0" />-->
+<!--      -->
+<!--  </xacro:kinect_v2>-->
   <xacro:include filename="$(find kinect_v2)/urdf/kinect_v2.urdf.xacro" />
-    <xacro:kinect_v2  parent="world">
-        <origin xyz="0.6 0 1.00"
-                rpy="0 1.57 0" />
+  <xacro:kinect_v2  parent="world">
+<!--    <origin xyz="0.6 0 1.00"-->
+<!--            rpy="0 1.57 0" /> -->
+    <origin xyz="1.0 0 0.8"
+            rpy="0 2.08 0" />
   </xacro:kinect_v2>
+  <!-- realsense d435 -->
+<!--  <xacro:include filename="$(find realsense2_description)/urdf/_d435.urdf.xacro" />-->
+<!--  <xacro:sensor_d435 name="camera" topics_ns="camera" parent="ee_link" publish_pointcloud="true">-->
+<!--              <origin xyz="-0.05 0 0.05"-->
+<!--                      rpy="0 -0.25 0" />-->
+<!--  </xacro:sensor_d435>-->
   <!-- kinect, ir, rgb sensor-->
 <!--   <xacro:include filename="$(find ur5_single_arm_tufts)/urdf/sensors/kinect2/common.xacro" />

File: ur5_single_arm_tufts/urdf/ur5_single_arm_with_table.urdf.xacro (robot description, xacro)
@@ -16,4 +16,24 @@
   <xacro:include filename="$(find ur5_single_arm_tufts)/urdf/cafe_table.urdf.xacro" />
   <xacro:cafe_table prefix="" />
+  <!-- cubes -->
+  <xacro:include filename="$(find ur5_single_arm_tufts)/urdf/cubes.urdf.xacro" />
+  <xacro:cubes prefix="1" />
+  <xacro:cubes prefix="2" />
+  <xacro:cubes prefix="3" />
+  <joint name="world_cube1_joint" type="fixed">
+    <parent link="world" />
+    <child link = "cube1" />
+    <origin xyz="0.4 -0.2 0.775" rpy="0.0 0.0 0.0" />
+  </joint>
+  <joint name="world_cube2_joint" type="fixed">
+    <parent link="world" />
+    <child link = "cube2" />
+    <origin xyz="0.4 0 0.775" rpy="0.0 0.0 0.0" />
+  </joint>
+  <joint name="world_cube3_joint" type="fixed">
+    <parent link="world" />
+    <child link = "cube3" />
+    <origin xyz="0.6 0.0 0.775" rpy="0.0 0.0 0.0" />
+  </joint>
     <!-- kinect -->
   <!--xacro:include filename="$(find ur5_single_arm_tufts)/urdf/sensors/kinect/kinect.urdf.xacro" />
@@ -23,5 +43,6 @@
   <xacro:include filename="$(find kinect_v2)/urdf/kinect_v2.urdf.xacro" />
     <xacro:kinect_v2  parent="world">
-        <origin xyz="0.6 0 1.00"
+<!--        <origin xyz="0.6 0 1.00"-->
+        <origin xyz="0.6 0 1.594"
                 rpy="0 1.57 0" />
   </xacro:kinect_v2>

Commit message: gpd

File: ur5_single_arm_tufts/urdf/ur5_single_arm.urdf.xacro (robot description, xacro)
@@ -10,6 +10,9 @@
   <xacro:include filename="$(find robotiq_85_description)/urdf/robotiq_85_gripper.urdf.xacro" />
   <!-- gripper -->
-  <xacro:robotiq_85_gripper prefix="" parent="ee_link" >
-    <origin xyz="0 0 0" rpy="0 0 0"/>
+<!--  <xacro:robotiq_85_gripper prefix="" parent="ee_link" >-->
+<!--    <origin xyz="0 0 0" rpy="0 0 0"/>-->
+<!--  </xacro:robotiq_85_gripper>-->
+  <xacro:robotiq_85_gripper prefix="" parent="wrist_3_link" >
+    <origin xyz="0.0 0.0823 0.0" rpy="0.0 0.0 1.5707" />
   </xacro:robotiq_85_gripper>
     <!-- kinect -->

Commit message: test for pointnetgpd

File: ur5_single_arm_tufts/urdf/ur5_single_arm.urdf.xacro (robot description, xacro)
@@ -38,15 +38,15 @@
   <xacro:include filename="$(find kinect_v2)/urdf/kinect_v2.urdf.xacro" />
   <xacro:kinect_v2  parent="world">
-<!--    <origin xyz="0.6 0 1.00"-->
-<!--            rpy="0 1.57 0" /> -->
+    <!--    <origin xyz="0.6 0 1.00"-->
+    <!--            rpy="0 1.57 0" /> -->
     <origin xyz="1.0 0 0.8"
             rpy="0 2.08 0" />
   </xacro:kinect_v2>
   <!-- realsense d435 -->
-<!--  <xacro:include filename="$(find realsense2_description)/urdf/_d435.urdf.xacro" />-->
-<!--  <xacro:sensor_d435 name="camera" topics_ns="camera" parent="ee_link" publish_pointcloud="true">-->
-<!--              <origin xyz="-0.05 0 0.05"-->
-<!--                      rpy="0 -0.25 0" />-->
-<!--  </xacro:sensor_d435>-->
+  <xacro:include filename="$(find realsense2_description)/urdf/_d435.urdf.xacro" />
+  <xacro:sensor_d435 name="camera" topics_ns="camera" parent="ee_link" publish_pointcloud="true">
+              <origin xyz="0.05 0 0.05"
+                      rpy="0 -0.08 0" />
+  </xacro:sensor_d435>
   <!-- kinect, ir, rgb sensor-->
 <!--   <xacro:include filename="$(find ur5_single_arm_tufts)/urdf/sensors/kinect2/common.xacro" />
@@ -63,4 +63,11 @@
     <child link = "base_link" />
     <origin xyz="0.0 0.0 0.0" rpy="0.0 0.0 0.0" />
+  </joint>
+  <link name="table_top"/>
+  <joint name="table_top_joint" type="fixed">
+    <parent link="world" />
+    <child link = "table_top" />
+    <!--  0.775-0.594  -->
+    <origin xyz="0.7 0 0.181" rpy="0.0 0.0 0.0" />
   </joint>
 <!--   <link name="table">

File: ur5_single_arm_tufts/urdf/ur5_single_arm_with_table.urdf.xacro (robot description, xacro)
@@ -47,4 +47,10 @@
                 rpy="0 1.57 0" />
   </xacro:kinect_v2>
+  <!-- realsense d435 -->
+  <xacro:include filename="$(find realsense2_description)/urdf/_d435.urdf.xacro" />
+  <xacro:sensor_d435 name="camera" topics_ns="camera" parent="ee_link" publish_pointcloud="true">
+    <origin xyz="-0.05 0 0.05"
+            rpy="0 -0.25 0" />
+  </xacro:sensor_d435>
   <!-- kinect, ir, rgb sensor-->
 <!--   <xacro:include filename="$(find ur5_single_arm_tufts)/urdf/sensors/kinect2/common.xacro" />
